File: Hardware/8eye line sensor.brd (EAGLE design)
At the start: 106.7 x 27.9 mm, 85 parts, among them U1 SX1509, U101 QRE1113, U102 QRE1113, U103 QRE1113, U104 QRE1113, U105 QRE1113, U106 QRE1113, U107 QRE1113, U108 QRE1113, U2 74AC125, U3 3.3V/150mA, U5 LM1117, U6 74AC125

Commit message: Ready for proto
Parts:
- removed LOGO3: SFE_LOGO_FLAME.3_INCH, SparkFun-Aesthetics:SFE_LOGO_FLAME_.3
- removed LOGO4: SFE_LOGO_NAME.2_INCH, SparkFun-Aesthetics:SFE_LOGO_NAME_.2
- removed STANDOFF1, STANDOFF2: STAND-OFF, SparkFun-Electromechanical:STAND-OFF
- added LOGO1: SFE_LOGO_NAME_FLAME.2_INCH, SparkFun-Aesthetics:SFE_LOGO_NAME_FLAME_.2
- moved LOGO5 3.08 mm to (8.81, 3.68)
- moved LOGO6 2.54 mm to (99.1, 5.08)
- moved LOGO2 0.79 mm to (63.7, 3.64)
Routing:
- net LED_BIAS: track 146.2 -> 147.6 mm
- net GND: vias 51 -> 52
Other:
- board text added: "00"
- board text added: "01"
- board text added: "0x3E"
- board text added: "0x3F"
- board text added: "0x70"
- board text added: "0x71"
- board text added: "10"
- board text added: "11"
- board text added: "2"
- board text added: "BRIGHTER"
- board text added: "C ADDR"
- board text added: "I"
- board text added: "IR"
- board text removed: "ADJ"
