File: Hardware/8eye line sensor.sch (EAGLE design)
At the start: 28 parts, among them U1 QRE1113, U10 QRE1113, U2 QRE1113, U3 QRE1113

Commit message: Layout commit
Parts:
- removed U$1: PCF8575C, SparkFun-DigitalIC:PCF8575C
- removed U1, U10, U2, U3: QRE1113, SparkFun-Sensors:QRE1113
- added C3: 1.0uF, SparkFun-Capacitors:1.0UF-16V-10%(0603)
- added D5, D6, D7, D8: GREEN, SparkFun-LED:LED-GREEN0603
- added JP1, JP2: (no value), SparkFun-Connectors:M04PTH
- added JP5: AVR_SPI_PRG_6PTH, SparkFun-Connectors:AVR_SPI_PRG_6PTH
- added LED2: Power, SparkFun-Nate:LED1206
- added R16: TRIMPOT-PTH-KNOB, SparkFun-Electromechanical:TRIMPOT-PTH-KNOB
- added R17, R18, R19, R20, R21, R22, R23, R24, R25, R26, R27, R28, R29, R30, R32: (no value), SparkFun-Passives:RESISTOR0603-RES
- added SJ1: A0, SparkFun:SOLDERJUMPER_2WAYS
- added SJ2: A1, SparkFun:SOLDERJUMPER_2WAYS
- added SJ3: A2, SparkFun:SOLDERJUMPER_2WAYS
- added U$3: 74ACT125D, SparkFun-Retired:74ACT125D
- added U101, U102, U103, U104, U105, U106, U107, U108: QRE1113, SparkFun-Sensors:QRE1113
- added U8: PCF8575C, SparkFun:PCF8575C
- R2: value (none) -> 330; device SparkFun-Passives:RESISTOR0603-RES -> SparkFun:RESISTOR0603-RES
Connections:
- removed net !ENB: U$2.A0
- removed net N$10: R8.1, U$2.O3
- removed net N$4: R5.1, U$2.O0
- removed net N$6: R6.1, U$2.O1
- removed net N$8: R7.1, U$2.O2
- new net !ENBLSB: R15.2, U$2.A0, U$2.A1, U$2.A2, U$2.A3
- new net !ENBMSB: R29.2, U$3.A0, U$3.A1, U$3.A2, U$3.A3
- new net A0: SJ1.2, U8.A0
- new net A1: SJ2.2, U8.A1
- new net A2: SJ3.2, U8.A2
- new net INT: U8.INT
- new net N$18: LED2.A, R2.1
- new net N$20: D5.A, R17.2
- new net N$22: D6.A, R18.2
- new net N$24: D7.A, R19.2
- new net N$26: D8.A, R20.2
- new net P10: JP2.4, U8.P10
- new net P11: JP2.3, U8.P11
- new net P12: JP2.2, U8.P12
- new net P13: JP2.1, U8.P13
- new net P14: JP1.4, U8.P14
- new net P15: JP1.3, U8.P15
- new net P16: JP1.2, U8.P16
- new net P17: JP1.1, U8.P17
- new net SCL: JP5.3, R30.1, U8.SCL
- new net SDA: JP5.1, R32.1, U8.SDA
- new net SEN1BUF: R8.1, U$2.O3, U8.PO0
- new net SEN2BUF: R7.1, U$2.O2, U8.PO1
- new net SEN3BUF: R5.1, U$2.O0, U8.PO2
- new net SEN4BUF: R6.1, U$2.O1, U8.PO3
- new net SEN5: R22.1, U$3.B3, U105.C
- new net SEN5BUF: R20.1, U$3.O3, U8.PO4
- new net SEN6: R26.1, U$3.B2, U106.C
- new net SEN6BUF: R19.1, U$3.O2, U8.PO5
- new net SEN7: R27.1, U$3.B0, U107.C
- new net SEN7BUF: R17.1, U$3.O0, U8.PO6
- new net SEN8: R28.1, U$3.B1, U108.C
- new net SEN8BUF: R18.1, U$3.O1, U8.PO7
- net GND: now also C3.2, D5.C, D6.C, D7.C, D8.C, JP5.6, LED2.C, R16.CW, R16.WIPER, R29.1, SJ1.3, SJ2.3, SJ3.3, U$3.GND, U101.E, U101.K, U102.E, U102.K, U103.E, U103.K, U104.E, U104.K, U105.E, U105.K, U106.E, U106.K, U107.E, U107.K, U108.E, U108.K, U8.GND; no longer R2.1, U$1.GND, U1.E, U1.K, U10.E, U10.K, U2.E, U2.K, U3.E, U3.K
- net LED_BIAS: now also R2.2, R21.1, R23.1, R24.1, R25.1
- net N$1: now also R16.CCW; no longer R2.2
- net N$12: now also U102.A; no longer U1.A
- net N$13: now also R23.2, U106.A; no longer U$2.B1
- net N$14: now also U103.A; no longer U2.A
- net N$15: now also R24.2, U107.A; no longer U$2.B2
- net N$16: now also U104.A; no longer U3.A
- net N$17: now also R25.2, U108.A; no longer U$2.B3
- net N$2: now also U101.A; no longer U10.A
- net N$3: now also R21.2, U105.A; no longer U$2.B0
- net SEN1: now also U$2.B3, U101.C; no longer U10.C
- net SEN2: now also U$2.B2, U102.C
- net SEN3: now also U$2.B0, U103.C
- net SEN4: now also U$2.B1, U104.C
- net VCC: now also C3.1, JP5.2, R22.2, R26.2, R27.2, R28.2, R30.2, R32.2, SJ1.1, SJ2.1, SJ3.1, U$3.VCC, U8.VCC; no longer U$1.VCC
Other:
- moved on the sheet: D1, D2, D3, D4, R10, R11, R12, R13, R14, R15, R2, R3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

Commit message: Shrunk PCB
Parts:
- removed IC1: (no value), SparkFun-PowerIC:V_REG_LM1117SOT223
- removed JP5: AVR_SPI_PRG_6PTH, SparkFun-Connectors:AVR_SPI_PRG_6PTH
- removed U$2, U$3: 74ACT125D, SparkFun-Retired:74ACT125D
- removed U8: PCF8575C, SparkFun:PCF8575C
- added C4: 2.2uF, SparkFun-Capacitors:2.2UF-10V-20%(0603)
- added C5, C6: 470pF, SparkFun-Capacitors:470PF-50V-5%(0603)SMD
- added FRAME2: FRAME-LEDGER, SparkFun-Aesthetics:FRAME-LEDGER
- added LOGO1: SFE_LOGO_NAME_FLAME.3_INCH, SparkFun-Aesthetics:SFE_LOGO_NAME_FLAME.3_INCH
- added R31: 100, SparkFun-Passives:RESISTOR0603-RES
- added U1: SX1509, SparkFun-DigitalIC:SX1509
- added U2, U4: 74ACT125D, SparkFun-Retired:74ACT125D
- added U3: 3.3V/150mA, SparkFun-PowerIC:V_REG_MIC52053.3V
- added U5: LM1117, SparkFun-PowerIC:V_REG_LM1117SOT223
- D1, D2, D3, D4, D5, D6, D7, D8: value GREEN -> Green; device SparkFun-LED:LED-GREEN0603 -> SparkFun-LED:LED-GREEN1206-BOTTOM
- JP1: value (none) -> FEMALE 2x3; device SparkFun-Connectors:M04PTH -> SparkFun-Connectors:M03X2FEMALE
- JP2: value (none) -> INT; device SparkFun-Connectors:M04PTH -> SparkFun-Connectors:M01PTH
- LED2: value Power -> Green; device SparkFun-Nate:LED1206 -> SparkFun-LED:LED-GREEN1206-BOTTOM
- R1: value (none) -> 4.7K
- R10, R12, R14, R22, R26, R27, R28, R4: value (none) -> 68K
- R11, R13, R21, R23, R24, R25, R3, R9: value (none) -> 100
- R15, R29, R30, R32: value (none) -> 10K
- R17, R18, R19, R20, R5, R6, R7, R8: value (none) -> 1K
- SJ3: value A2 -> A1; device SparkFun:SOLDERJUMPER_2WAYS -> SparkFun-Passives:JUMPER-PAD-3-NC_BY_PASTE
Connections:
- removed net A2: SJ3.2, U8.A2
- removed net P10: JP2.4, U8.P10
- removed net P11: JP2.3, U8.P11
- removed net P12: JP2.2, U8.P12
- removed net P13: JP2.1, U8.P13
- removed net P14: JP1.4, U8.P14
- removed net P15: JP1.3, U8.P15
- removed net P16: JP1.2, U8.P16
- removed net P17: JP1.1, U8.P17
- new net I2C_PWR: C3.1, C4.1, R31.1, SJ1.1, SJ2.1, U1.VCC1, U1.VCC2, U1.VDDM, U3.OUT
- new net N$4: R30.2, SJ3.1
- new net N$6: C5.1, U3.BP
- new net N$8: R32.2, SJ3.3
- new net ~RESET: C6.1, R31.2, U1.!RESET
- net !ENBLSB: now also U2.A0, U2.A1, U2.A2, U2.A3; no longer U$2.A0, U$2.A1, U$2.A2, U$2.A3
- net !ENBMSB: now also U4.A0, U4.A1, U4.A2, U4.A3; no longer U$3.A0, U$3.A1, U$3.A2, U$3.A3
- net A0: now also U1.ADDR0; no longer U8.A0
- net A1: now also U1.ADDR1; no longer U8.A1
- net GND: now also C4.2, C5.2, C6.2, JP1.1, JP1.2, U1.GND, U2.GND, U3.GND, U4.GND; no longer JP5.6, SJ3.3, U$2.GND, U$3.GND, U8.GND
- net INT: now also JP2.1, U1.!INT; no longer U8.INT
- net LED_BIAS: now also U5.OUT, U5.OUT@1; no longer IC1.OUT, IC1.OUT@1
- net N$1: now also U5.ADJ; no longer IC1.ADJ
- net SCL: now also JP1.5, U1.SCL; no longer JP5.3, U8.SCL
- net SDA: now also JP1.6, U1.SDA; no longer JP5.1, U8.SDA
- net SEN1: now also U2.B0; no longer U$2.B3
- net SEN1BUF: now also R5.1, U1.I/O[0], U2.O0; no longer R8.1, U$2.O3, U8.PO0
- net SEN2: now also U2.B1; no longer U$2.B2
- net SEN2BUF: now also R6.1, U1.I/O[1], U2.O1; no longer R7.1, U$2.O2, U8.PO1
- net SEN3: now also U2.B2; no longer U$2.B0
- net SEN3BUF: now also R7.1, U1.I/O[2], U2.O2; no longer R5.1, U$2.O0, U8.PO2
- net SEN4: now also U2.B3; no longer U$2.B1
- net SEN4BUF: now also R8.1, U1.I/O[3], U2.O3; no longer R6.1, U$2.O1, U8.PO3
- net SEN5: now also U4.B0; no longer U$3.B3
- net SEN5BUF: now also R17.1, U1.I/O[4], U4.O0; no longer R20.1, U$3.O3, U8.PO4
- net SEN6: now also U4.B1; no longer U$3.B2
- net SEN6BUF: now also R18.1, U1.I/O[5], U4.O1; no longer R19.1, U$3.O2, U8.PO5
- net SEN7: now also U4.B2; no longer U$3.B0
- net SEN7BUF: now also R19.1, U1.I/O[6], U4.O2; no longer R17.1, U$3.O0, U8.PO6
- net SEN8: now also U4.B3; no longer U$3.B1
- net SEN8BUF: now also R20.1, U1.I/O[7], U4.O3; no longer R18.1, U$3.O1, U8.PO7
- net VCC: now also JP1.3, JP1.4, SJ3.2, U2.VCC, U3.EN, U3.IN, U4.VCC, U5.IN; no longer C3.1, IC1.IN, JP5.2, R30.2, R32.2, SJ1.1, SJ2.1, SJ3.1, U$2.VCC, U$3.VCC, U8.VCC
Other:
- note added: "Buffers"
- note added: "High order nibble"
- note added: "I2C/RedBot Interface"
- note added: "Low order nibble"
- note added: "Marshall Taylor"
- note added: "Power"
- note added: "Sensors"
- note added: "V02"
- moved on the sheet: C1, C2, C3, D1, D2, D3, D4, D5, D6, D7, D8, R1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

Commit message: logos and 47 measures and t_place added, Oh my!
Parts:
- removed LOGO1: SFE_LOGO_NAME_FLAME.3_INCH, SparkFun-Aesthetics:SFE_LOGO_NAME_FLAME.3_INCH
- added FID1, FID2: FIDUCIALUFIDUCIAL, SparkFun-Aesthetics:FIDUCIALUFIDUCIAL
- added LOGO2, LOGO4: SFE_LOGO_NAME.2_INCH, SparkFun-Aesthetics:SFE_LOGO_NAME.2_INCH
- added LOGO3, LOGO5: SFE_LOGO_FLAME.3_INCH, SparkFun-Aesthetics:SFE_LOGO_FLAME.3_INCH
- added LOGO6: OSHW-LOGOS, SparkFun-Aesthetics:OSHW-LOGOS
- added STANDOFF1, STANDOFF2: STAND-OFF, SparkFun-Electromechanical:STAND-OFF
Changed lines of the file:
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@@
 <part name="FRAME2" library="SparkFun-Aesthetics" deviceset="FRAME-LEDGER" device=""/>
 <part name="JP2" library="SparkFun-Connectors" deviceset="M01" device="PTH" value="INT"/>
-<part name="LOGO1" library="SparkFun-Aesthetics" deviceset="SFE_LOGO_NAME_FLAME" device=".3_INCH"/>
+<part name="LOGO2" library="SparkFun-Aesthetics" deviceset="SFE_LOGO_NAME" device=".2_INCH" value="SFE_LOGO_NAME.2_INCH"/>
+<part name="LOGO3" library="SparkFun-Aesthetics" deviceset="SFE_LOGO_FLAME" device=".3_INCH"/>
+<part name="LOGO4" library="SparkFun-Aesthetics" deviceset="SFE_LOGO_NAME" device=".2_INCH" value="SFE_LOGO_NAME.2_INCH"/>
+<part name="LOGO5" library="SparkFun-Aesthetics" deviceset="SFE_LOGO_FLAME" device=".3_INCH"/>
+<part name="LOGO6" library="SparkFun-Aesthetics" deviceset="OSHW-LOGO" device="S"/>
+<part name="FID1" library="SparkFun-Aesthetics" deviceset="FIDUCIAL" device="UFIDUCIAL"/>
+<part name="FID2" library="SparkFun-Aesthetics" deviceset="FIDUCIAL" device="UFIDUCIAL"/>
+<part name="STANDOFF1" library="SparkFun-Electromechanical" deviceset="STAND-OFF" device=""/>
+<part name="STANDOFF2" library="SparkFun-Electromechanical" deviceset="STAND-OFF" device=""/>
 </parts>
 <sheets>
@@
 <instance part="FRAME2" gate="G$2" x="330.2" y="0"/>
 <instance part="JP2" gate="G$1" x="50.8" y="40.64"/>
-<instance part="LOGO1" gate="G$1" x="332.74" y="48.26"/>
+<instance part="LOGO2" gate="G$1" x="447.04" y="116.84"/>
+<instance part="LOGO3" gate="G$1" x="452.12" y="96.52"/>
+<instance part="LOGO4" gate="G$1" x="538.48" y="119.38"/>
+<instance part="LOGO5" gate="G$1" x="543.56" y="96.52"/>
+<instance part="LOGO6" gate="G$1" x="469.9" y="73.66"/>
+<instance part="FID1" gate="G$1" x="502.92" y="45.72"/>
+<instance part="FID2" gate="G$1" x="518.16" y="48.26"/>
+<instance part="STANDOFF1" gate="G$1" x="541.02" y="48.26"/>
+<instance part="STANDOFF2" gate="G$1" x="558.8" y="45.72"/>
 </instances>
 <busses>

Commit message: about ready for proto submit
Other:
- note added: "A1:A0 00 01 10 11"
- note added: "I2C Address 0x3E (0111110b) 0x3F (0111111b) 0x70 (1110000b) 0x71 (1110001b)"
- note added: "I2C Expander"
- note added: "Open SJ3 to disconnect I2C pull-up resistors"
- note added: "Possible I2C addresses"
- note added: "RedBot Interface"
- note added: "Set I2C addres with SJ1 and SJ2"
- note added: "Supply +5V"
- note removed: "I2C/RedBot Interface"
- moved on the sheet: C3, C6, JP1, JP2, R30, R31, R32, SJ1, SJ2, SJ3, U1

Commit message: fixed for QC
Parts:
- added STANDOFF3, STANDOFF4: STAND-OFF, SparkFun-Electromechanical:STAND-OFF
- R1: device SparkFun-Passives:RESISTOR0603-RES -> SparkFun-Resistors:4.7KOHM-1/10W-1%(0603)
- R10, R12, R14, R22, R26, R27, R28, R4: device SparkFun-Passives:RESISTOR0603-RES -> SparkFun-Resistors:68.1KOHM1/10W1%(0603)
- R11, R13, R21, R23, R24, R25, R3, R31, R9: device SparkFun-Passives:RESISTOR0603-RES -> SparkFun-Resistors:100OHM-1/10W-1%(0603)
- R15, R29, R30, R32: device SparkFun-Passives:RESISTOR0603-RES -> SparkFun-Resistors:10KOHM-1/10W-1%(0603)0603
- R16: value TRIMPOT-PTH-KNOB -> TSR-3386
- R17, R18, R19, R20, R5, R6, R7, R8: device SparkFun-Passives:RESISTOR0603-RES -> SparkFun-Resistors:1KOHM-1/10W-1%(0603)
- R2: value 330 -> 33OHM; device SparkFun:RESISTOR0603-RES -> SparkFun-Resistors:33OHM1/10W1%(0603)
- U2, U4: value 74ACT125D -> IC-08880
Connections:
- removed net SEN8: R28.1, U108.C, U4.B3
- removed net SEN8BUF: R20.1, U1.I/O[7], U4.O3
- new net SEN0: R4.1, U101.C, U2.B0
- new net SEN0BUF: R5.1, U1.I/O[0], U2.O0
- net SEN1: now also R10.1, U102.C, U2.B1; no longer R4.1, U101.C, U2.B0
- net SEN1BUF: now also R6.1, U1.I/O[1], U2.O1; no longer R5.1, U1.I/O[0], U2.O0
- net SEN2: now also R12.1, U103.C, U2.B2; no longer R10.1, U102.C, U2.B1
- net SEN2BUF: now also R7.1, U1.I/O[2], U2.O2; no longer R6.1, U1.I/O[1], U2.O1
- net SEN3: now also R14.1, U104.C, U2.B3; no longer R12.1, U103.C, U2.B2
- net SEN3BUF: now also R8.1, U1.I/O[3], U2.O3; no longer R7.1, U1.I/O[2], U2.O2
- net SEN4: now also R22.1, U105.C, U4.B0; no longer R14.1, U104.C, U2.B3
- net SEN4BUF: now also R17.1, U1.I/O[4], U4.O0; no longer R8.1, U1.I/O[3], U2.O3
- net SEN5: now also R26.1, U106.C, U4.B1; no longer R22.1, U105.C, U4.B0
- net SEN5BUF: now also R18.1, U1.I/O[5], U4.O1; no longer R17.1, U1.I/O[4], U4.O0
- net SEN6: now also R27.1, U107.C, U4.B2; no longer R26.1, U106.C, U4.B1
- net SEN6BUF: now also R19.1, U1.I/O[6], U4.O2; no longer R18.1, U1.I/O[5], U4.O1
- net SEN7: now also R28.1, U108.C, U4.B3; no longer R27.1, U107.C, U4.B2
- net SEN7BUF: now also R20.1, U1.I/O[7], U4.O3; no longer R19.1, U1.I/O[6], U4.O2
Other:
- note added: "Note: Footprint for IC-08880 will be updated after first proto order for U2 and U4"

Commit message: fixed half the issues
Parts:
- removed U4: IC-08880, SparkFun-Retired:74ACT125D
- added C7: 2.2uF, SparkFun-Capacitors:2.2UF-10V-20%(0603)
- added SJ5: JUMPER-PAD-3-2OF3_NC_BY_TRACE_SMALL, SparkFun-Passives:JUMPER-PAD-3-2OF3_NC_BY_TRACE_SMALL
- added U6: 74AC125, SparkFun-DigitalIC:74AC125DG125
- SJ1, SJ2: device SparkFun:SOLDERJUMPER_2WAYS -> SparkFun-Passives:JUMPER-PAD-3-2OF3_NC_BY_PASTE
- SJ3: device SparkFun-Passives:JUMPER-PAD-3-NC_BY_PASTE -> SparkFun-Passives:JUMPER-PAD-3-NC_BY_TRACE
- U2: value IC-08880 -> 74AC125; device SparkFun-Retired:74ACT125D -> SparkFun-DigitalIC:74AC125DG125
Connections:
- new net N$19: SJ3.2, SJ5.2
- net !ENBLSB: now also U2G0.!EN, U2G1.!EN, U2G2.!EN, U2G3.!EN; no longer U2.A0, U2.A1, U2.A2, U2.A3
- net !ENBMSB: now also U6G0.!EN, U6G1.!EN, U6G2.!EN, U6G3.!EN; no longer U4.A0, U4.A1, U4.A2, U4.A3
- net GND: now also C7.2, U2PWR.P$V-, U6PWR.P$V-; no longer U2.GND, U4.GND
- net I2C_PWR: now also C7.1, SJ5.3; no longer U1.VCC1
- net SEN0: now also U2G0.D; no longer U2.B0
- net SEN0BUF: now also U2G0.Q; no longer U2.O0
- net SEN1: now also U2G1.D; no longer U2.B1
- net SEN1BUF: now also U2G1.Q; no longer U2.O1
- net SEN2: now also U2G2.D; no longer U2.B2
- net SEN2BUF: now also U2G2.Q; no longer U2.O2
- net SEN3: now also U2G3.D; no longer U2.B3
- net SEN3BUF: now also U2G3.Q; no longer U2.O3
- net SEN4: now also U6G0.D; no longer U4.B0
- net SEN4BUF: now also U6G0.Q; no longer U4.O0
- net SEN5: now also U6G1.D; no longer U4.B1
- net SEN5BUF: now also U6G1.Q; no longer U4.O1
- net SEN6: now also U6G2.D; no longer U4.B2
- net SEN6BUF: now also U6G2.Q; no longer U4.O2
- net SEN7: now also U6G3.D; no longer U4.B3
- net SEN7BUF: now also U6G3.Q; no longer U4.O3
- net VCC: now also SJ5.1, U1.VCC1, U2PWR.P$V+, U6PWR.P$V+; no longer SJ3.2, U2.VCC, U4.VCC
Other:
- note added: "V03"
- note removed: "Note: Footprint for IC-08880 will be updated after first proto order for U2 and U4"
- note removed: "V02"
- moved on the sheet: D1, D2, D3, D4, D5, D6, D7, D8, JP1, R15, R17, R18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

Commit message: ready for review of prototype 2 (v03)
Parts:
- added R33, R34: 4.7K, SparkFun-Resistors:4.7KOHM-1/10W-1%(0603)
Connections:
- new net N$10: R34.2, SJ2.1
- new net N$21: R33.2, SJ1.1
- net I2C_PWR: now also R33.1, R34.1; no longer SJ1.1, SJ2.1
Other:
- moved on the sheet: D1, D2, D3, D4, D5, D6, D7, D8, R17, R18, R19, R20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

Commit message: Ready for proto
Parts:
- removed LOGO3: SFE_LOGO_FLAME.3_INCH, SparkFun-Aesthetics:SFE_LOGO_FLAME.3_INCH
- removed LOGO4: SFE_LOGO_NAME.2_INCH, SparkFun-Aesthetics:SFE_LOGO_NAME.2_INCH
- removed STANDOFF1, STANDOFF2: STAND-OFF, SparkFun-Electromechanical:STAND-OFF
- added LOGO1: SFE_LOGO_NAME_FLAME.2_INCH, SparkFun-Aesthetics:SFE_LOGO_NAME_FLAME.2_INCH
Changed lines of the file:
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@@
 <part name="JP2" library="SparkFun-Connectors" deviceset="M01" device="PTH" value="INT"/>
 <part name="LOGO2" library="SparkFun-Aesthetics" deviceset="SFE_LOGO_NAME" device=".2_INCH" value="SFE_LOGO_NAME.2_INCH"/>
-<part name="LOGO3" library="SparkFun-Aesthetics" deviceset="SFE_LOGO_FLAME" device=".3_INCH"/>
-<part name="LOGO4" library="SparkFun-Aesthetics" deviceset="SFE_LOGO_NAME" device=".2_INCH" value="SFE_LOGO_NAME.2_INCH"/>
 <part name="LOGO5" library="SparkFun-Aesthetics" deviceset="SFE_LOGO_FLAME" device=".3_INCH"/>
 <part name="LOGO6" library="SparkFun-Aesthetics" deviceset="OSHW-LOGO" device="S"/>
 <part name="FID1" library="SparkFun-Aesthetics" deviceset="FIDUCIAL" device="UFIDUCIAL"/>
 <part name="FID2" library="SparkFun-Aesthetics" deviceset="FIDUCIAL" device="UFIDUCIAL"/>
-<part name="STANDOFF1" library="SparkFun-Electromechanical" deviceset="STAND-OFF" device=""/>
-<part name="STANDOFF2" library="SparkFun-Electromechanical" deviceset="STAND-OFF" device=""/>
 <part name="STANDOFF3" library="SparkFun-Electromechanical" deviceset="STAND-OFF" device=""/>
 <part name="STANDOFF4" library="SparkFun-Electromechanical" deviceset="STAND-OFF" device=""/>
@@
 <part name="R33" library="SparkFun-Resistors" deviceset="4.7KOHM-1/10W-1%(0603)" device="" value="4.7K"/>
 <part name="R34" library="SparkFun-Resistors" deviceset="4.7KOHM-1/10W-1%(0603)" device="" value="4.7K"/>
+<part name="LOGO1" library="SparkFun-Aesthetics" deviceset="SFE_LOGO_NAME_FLAME" device=".2_INCH"/>
 </parts>
 <sheets>
@@
 <instance part="FRAME2" gate="G$2" x="330.2" y="0"/>
 <instance part="JP2" gate="G$1" x="63.5" y="40.64"/>
-<instance part="LOGO2" gate="G$1" x="355.6" y="76.2"/>
-<instance part="LOGO3" gate="G$1" x="342.9" y="76.2"/>
-<instance part="LOGO4" gate="G$1" x="355.6" y="63.5"/>
-<instance part="LOGO5" gate="G$1" x="342.9" y="63.5"/>
-<instance part="LOGO6" gate="G$1" x="355.6" y="50.8"/>
-<instance part="FID1" gate="G$1" x="368.3" y="50.8"/>
-<instance part="FID2" gate="G$1" x="381" y="50.8"/>
-<instance part="STANDOFF1" gate="G$1" x="393.7" y="50.8"/>
-<instance part="STANDOFF2" gate="G$1" x="401.32" y="50.8"/>
-<instance part="STANDOFF3" gate="G$1" x="408.94" y="50.8"/>
-<instance part="STANDOFF4" gate="G$1" x="416.56" y="50.8"/>
+<instance part="LOGO2" gate="G$1" x="337.82" y="45.72"/>
+<instance part="LOGO5" gate="G$1" x="406.4" y="50.8"/>
+<instance part="LOGO6" gate="G$1" x="411.48" y="76.2"/>
+<instance part="FID1" gate="G$1" x="403.86" y="40.64"/>
+<instance part="FID2" gate="G$1" x="411.48" y="40.64"/>
+<instance part="STANDOFF3" gate="G$1" x="419.1" y="40.64"/>
+<instance part="STANDOFF4" gate="G$1" x="426.72" y="40.64"/>
 <instance part="U6" gate="G0" x="340.36" y="248.92"/>
 <instance part="U6" gate="G1" x="340.36" y="233.68"/>
@@
 <instance part="R33" gate="G$1" x="170.18" y="40.64" rot="R270"/>
 <instance part="R34" gate="G$1" x="149.86" y="40.64" rot="R270"/>
+<instance part="LOGO1" gate="G$1" x="339.09" y="58.928"/>
 </instances>
 <busses>
