File: Hardware/SparkFun Line Follower Array.brd (EAGLE design)
At the start: 106.7 x 27.9 mm, 82 parts, among them Q1 MOSFET-NCHANNEL2N7002PW, U1 SX1509, U101 QRE1113, U102 QRE1113, U103 QRE1113, U104 QRE1113, U105 QRE1113, U106 QRE1113, U107 QRE1113, U108 QRE1113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

Commit message: Renamed project
Parts:
- moved LOGO6 3.81 mm to (102.9, 5.08)
Other:
- board text added: "Line Follower Array"
- board text removed: "RedBot Sensor Bar"
Changed lines of the file:
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@@
 <grid distance="0.1" unitdist="inch" unit="inch" style="lines" multiple="1" display="yes" altdistance="0.005" altunitdist="inch" altunit="inch"/>
 <layers>
-<layer number="1" name="Top" color="4" fill="1" visible="yes" active="yes"/>
+<layer number="1" name="Top" color="4" fill="1" visible="no" active="yes"/>
 <layer number="2" name="Route2" color="1" fill="3" visible="no" active="no"/>
 <layer number="3" name="Route3" color="4" fill="3" visible="no" active="no"/>
@@
 <layer number="19" name="Unrouted" color="6" fill="1" visible="yes" active="yes"/>
 <layer number="20" name="Dimension" color="15" fill="1" visible="yes" active="yes"/>
-<layer number="21" name="tPlace" color="15" fill="1" visible="yes" active="yes"/>
+<layer number="21" name="tPlace" color="15" fill="1" visible="no" active="yes"/>
 <layer number="22" name="bPlace" color="14" fill="1" visible="yes" active="yes"/>
 <layer number="23" name="tOrigins" color="15" fill="1" visible="no" active="yes"/>
@@
 <wire x1="106.68" y1="27.94" x2="0" y2="27.94" width="0.2032" layer="20"/>
 <wire x1="0" y1="27.94" x2="0" y2="0" width="0.2032" layer="20"/>
-<text x="2.54" y="1.42875" size="1.778" layer="21" font="vector" ratio="15">RedBot Sensor Bar</text>
+<text x="66.675" y="8.03275" size="1.778" layer="21" font="vector" ratio="15">Line Follower Array</text>
 <text x="8.5725" y="22.86" size="1.778" layer="21" font="vector" ratio="15" align="center">b7</text>
 <text x="22.06625" y="22.86" size="1.778" layer="21" font="vector" ratio="15" align="center">b6</text>
@@
 <element name="LOGO2" library="SparkFun-Aesthetics" package="SFE_LOGO_NAME_.2" value="SFE_LOGO_NAME.2_INCH" x="63.6905" y="3.6449" rot="MR0"/>
 <element name="LOGO5" library="SparkFun-Aesthetics" package="SFE_LOGO_FLAME_.3" value="SFE_LOGO_FLAME.3_INCH" x="8.80745" y="3.683" rot="MR0"/>
-<element name="LOGO6" library="SparkFun-Aesthetics" package="OSHW-LOGO-S" value="OSHW-LOGOS" x="99.06" y="5.08"/>
+<element name="LOGO6" library="SparkFun-Aesthetics" package="OSHW-LOGO-S" value="OSHW-LOGOS" x="102.87" y="5.08"/>
 <element name="FID1" library="SparkFun-Aesthetics" package="MICRO-FIDUCIAL" value="FIDUCIALUFIDUCIAL" x="2.54" y="2.54" rot="MR0"/>
 <element name="FID2" library="SparkFun-Aesthetics" package="MICRO-FIDUCIAL" value="FIDUCIALUFIDUCIAL" x="104.14" y="20.32" rot="MR0"/>
