File: Production/SparkFun_Line_Follower_Array_Panel_v10.brd (EAGLE design)
At the start: 120.4 x 297.7 mm, 813 parts, among them Q1 MOSFET-NCHANNEL2N7002PW, Q10 MOSFET-NCHANNEL2N7002PW, Q2 MOSFET-NCHANNEL2N7002PW, Q3 MOSFET-NCHANNEL2N7002PW, Q4 MOSFET-NCHANNEL2N7002PW, Q5 MOSFET-NCHANNEL2N7002PW, Q6 MOSFET-NCHANNEL2N7002PW, Q7 MOSFET-NCHANNEL2N7002PW, Q8 MOSFET-NCHANNEL2N7002PW, Q9 MOSFET-NCHANNEL2N7002PW, U1 SX1509, U10 QRE1113, U100 QRE1113, U101 QRE1113, U102 QRE1113, U103 QRE1113, U104 QRE1113, U105 QRE1113, U106 QRE1113, U107 QRE1113, U108 QRE1113, U109 QRE1113, U11 QRE1113, U110 QRE1113, U111 QRE1113, U112 QRE1113, U113 QRE1113, U114 SX1509, U115 3.3V/150mA, U116 74AC125, U117 74AC125, U118 LM1117, U119 QRE1113, U12 QRE1113, U120 QRE1113, U121 QRE1113, U122 QRE1113, U123 QRE1113, U124 QRE1113, U125 QRE1113, U126 QRE1113, U127 SX1509, U128 3.3V/150mA, U129 74AC125, U13 QRE1113, U130 74AC125, U14 QRE1113, U15 SX1509, U16 3.3V/150mA, U17 74AC125, U18 74AC125, U19 LM1117, U2 74AC125, U20 QRE1113, U21 QRE1113, U22 QRE1113, U23 QRE1113, U24 QRE1113, U25 QRE1113, U26 QRE1113, U27 QRE1113, U28 SX1509, U29 3.3V/150mA, U3 3.3V/150mA, U30 74AC125, U31 74AC125, U32 LM1117, U33 QRE1113, U34 QRE1113, U35 QRE1113, U36 QRE1113, U37 QRE1113, U38 QRE1113, U39 QRE1113, U4 LM1117, U40 QRE1113, U41 SX1509, U42 3.3V/150mA, U43 74AC125, U44 74AC125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

Commit message: created panel v10
Parts:
- moved R319 20.3 mm to (68.8, 299.7)
- moved C73 20.3 mm to (19.2, 290.7)
- moved C74 20.3 mm to (19.2, 292.3)
- moved C75 20.3 mm to (52.6, 300.7)
- moved C76 20.3 mm to (97.0, 294.0)
- moved C77 20.3 mm to (91.9, 293.4)
- moved C78 20.3 mm to (61.8, 301.3)
- moved C79 20.3 mm to (98.3, 294.0)
- moved C80 20.3 mm to (18.6, 294.2)
- moved D82 20.3 mm to (13.2, 298.4)
- moved D83 20.3 mm to (53.8, 303.5)
- moved D84 20.3 mm to (41.1, 303.5)
- moved D85 20.3 mm to (28.4, 303.5)
- moved D86 20.3 mm to (15.7, 303.5)
- moved D87 20.3 mm to (104.6, 303.5)
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Other:
- board size 120.4 x 297.7 mm -> 120.4 x 318 mm
- board text added: "Route Out"
